File: Trapezoid_Terminal/Interface Board/Entrex Trapezoid Interface Board v23.kicad_pcb (KiCad board)
At the start: 2 copper layers, 169.1 x 191 mm, 101 parts, among them P15 Conn_02x40_Odd_Even_Shielded, SW1 SW_DIP_x08

Commit message: checkin
Connections:
- UA7 pad 3: u7-13 -> /XX(UA7P3)
Routing:
- net u7-13: track 280.8 -> 272.1 mm
