File: Trapezoid_Terminal/Interface Board/Entrex Trapezoid Interface Board v23.kicad_sch (KiCad schematic)
At the start: 103 parts, among them P15 Conn_02x40_Odd_Even_Shielded, SW1 SW_DIP_x08

Commit message: checkin
Parts:
- removed C101: 0.1UF-0603-25V-5%, Capacitor_THT:C_Disc_D4.7mm_W2.5mm_P5.00mm, symbol SparkFun-Capacitors:0.1UF-0603-25V-5%
- removed DPLX_sw_SG1, DPLX_sw_SG2: SW_SPDT, symbol Switch:SW_SPDT
- removed R0, R1000: 330R, Resistor_THT:R_Axial_DIN0207_L6.3mm_D2.5mm_P10.16mm_Horizontal, symbol SamacSys_Parts:YR1B24K9CC
- removed R101: 150R, Resistor_THT:R_Axial_DIN0207_L6.3mm_D2.5mm_P10.16mm_Horizontal, symbol SamacSys_Parts:YR1B24K9CC
- removed unit 1 of UB6
- removed unit 3 of UB6
- removed unit 4 of UB6
- removed unit 3 of UB8
- removed unit 2 of UB8
- removed unit 1 of UB8
- removed unit 2 of UD7
- removed unit 3 of UD7
- removed unit 4 of UD7
- removed unit 1 of UD7
- removed unit 4 of UD8
- removed unit 1 of UD8
- removed unit 2 of UD8
- removed unit 5 of UD8
- removed unit 3 of UD8
- removed unit 6 of UD8
- added C29: 0.1UF-0603-25V-5%, Capacitor_THT:C_Disc_D4.7mm_W2.5mm_P5.00mm, symbol SparkFun-Capacitors:0.1UF-0603-25V-5%
- added R1: 10K, Resistor_THT:R_Axial_DIN0207_L6.3mm_D2.5mm_P10.16mm_Horizontal, symbol SamacSys_Parts:YR1B24K9CC
- added R24: 330R, Resistor_THT:R_Axial_DIN0207_L6.3mm_D2.5mm_P10.16mm_Horizontal, symbol SamacSys_Parts:YR1B24K9CC
- added R25: 150R, Resistor_THT:R_Axial_DIN0207_L6.3mm_D2.5mm_P10.16mm_Horizontal, symbol SamacSys_Parts:YR1B24K9CC
- added UA9, UB2, UC9: SN74LS00N, Package_DIP:DIP-14_W7.62mm, symbol 74xx:74LS00
- added UB1, UD4: SN74LS08N, Package_DIP:DIP-14_W7.62mm, symbol 74xx:74LS08
- added UB9: SN74LS74AN, Package_DIP:DIP-14_W7.62mm, symbol 74xx:74LS74
- added UD2: SN74LS04N, Package_DIP:DIP-14_W7.62mm, symbol 74xx:74LS04
- R19: value 10K -> 330R
Connections:
- net P15_45 is gone; now on net CG1_PIN_N: P15.45 (Pin_45), UD5.5 (1B)
- net u36_13 is gone; now on net VCC: UA1.13 (DS2), UA2.13 (DS2)
- net GND: now also C29.2
- net P15_14: no longer R3.2, UC1.6 (In3)
- net P15_16: no longer R2.2, UC1.10 (In4)
- net P15_18: no longer R4.2, UC1.12 (In5)
- net P15_20: no longer R5.2, UC1.4 (In2)
- net P15_22: no longer R6.1, UC1.14 (In6)
- net P15_24: no longer R7.1, UC1.2 (In1)
- net P15_64: no longer UC2.13, UE7.12
- net P15_66: no longer UC2.11, UF6.3
- net VCC: now also R1.2; no longer R19.2
- net XX(UB5P11): now also UB9.11 (C)
- net XX(UB5P9): now also UB9.9 (Q)
- net XX(UB8P12): no longer UB8.12
- net XX(UC7P8): no longer UC7.8 (~{Q})
- net XX(UD7P2): now also UD4.2
- net XX(UE3P10): no longer UE3.10 (~{S})
- net u10_11: now also UD4.11
- net u4_10: now also UD2.10
- net u4_12: now also UD2.12; no longer UD5.3 (1STRB), UD6.13 (2STRB)
- net u4_2: now also UD2.2, UD4.1
- net D1P1: no longer names the net of UC2.6, UC6.4
- net P15_10 renamed read_printer_status_reg
- net P15_11 renamed D4_in
- net D4_in: no longer UA2.16 (DI5)
- net P15_12 renamed read_latch_strobe
- net read_latch_strobe: now also UB1.12; no longer UC3.1 (M), UC3.2 (N)
- net P15_13 renamed D3_in
- net P15_15 renamed D2_in
- net P15_17 renamed D1_in
- net P15_19 renamed D0_in
- net P15_21 renamed D0_out
- net D0_out: no longer UE4.13 (Out6)
- net P15_23 renamed D1_out
- net P15_25 renamed D2_out
- net P15_27 renamed D3_out
- net P15_29 renamed D4_out
- net P15_31 renamed D5_out
- net P15_33 renamed D6_out
- net P15_35 renamed D7_out
- net P15_37 renamed CG1_PIN_N
- net P15_38 renamed CG1_PIN_B
- net P15_39 renamed CG1_PIN_A
- net P15_40 renamed CG1_PIN_F
- net P15_41 renamed CG1_PIN_J
- net P15_42 renamed CG1_PIN_P
- net P15_43 renamed CG1_PIN_R
- net P15_44: no longer names the net of UD5.9 (2A)
- net P15_44: no longer P15.44 (Pin_44)
- net P15_46: no longer names the net of UD5.11 (2B)
- net P15_46: no longer P15.46 (Pin_46)
- net P15_47 renamed CG_SEL2
- net CG_SEL2: now also UD2.13
- net P15_48 renamed CG_SEL1
- net CG_SEL1: now also UD2.1
- net P15_49 renamed CG2_PIN_H
- net P15_5 renamed D7_in
- net P15_50 renamed CG2_PIN_D
- net P15_51 renamed CG2_PIN_R
- net P15_52 renamed CG2_PIN_P
- net P15_53 renamed CG2_PIN_J
- net P15_54 renamed CG2_PIN_N
- net P15_55 renamed CG2_PIN_C
- net P15_56 renamed CG2_PIN_B
- net P15_57 renamed CG2_PIN_A
- net P15_58 renamed CG2_PIN_F
- net P15_59 renamed D7_in9
- net P15_7 renamed D6_in
- net P15_70 renamed D6_in0
- net P15_71 renamed D6_in1
- net P15_72 renamed D6_in2
- net P15_75 renamed D6_in5
- net P15_76 renamed D6_in6
- net P15_77 renamed D6_in7
- net P15_78 renamed D6_in8
- net P15_79 renamed D6_in9
- net D6_in9: now also UB1.9
- net P15_8 renamed read_status_latch
- net P15_9 renamed D5_in
- net D5_in: no longer UA5.4 (J)
- net U44P12: no longer names the net of UC6.6
- net U44P12: now also UB1.1
- net UA1_17: no longer names the net of UA1.17 (DO6), UD1.11
- net UA1_8: no longer names the net of UA1.8 (DO3), UD1.1
- net XX(UA2P11): no longer names the net of UA2.11 (Strobe)
- net XX(UC7P5): no longer names the net of UC7.5 (Q)
- net XX(UD5P14): no longer names the net of UD5.14 (2YP_(Sink))
- net XX(UD5P2): no longer names the net of UD5.2 (1YP_(Sink))
- net XX(UD6P14): no longer names the net of UD6.14 (2YP_(Sink))
- net XX(UD6P2): no longer names the net of UD6.2 (1YP_(Sink))
- net XX(UF4P6): no longer names the net of UF4.6 (~{Q})
- net XXUE6P14: no longer names the net of UE6.14 (2YP_(Sink))
- net XXUE6P2: no longer names the net of UE6.2 (1YP_(Sink))
- net u10_3: no longer names the net of UD6.3 (1STRB)
- net u10_3: now also UD4.3
- net u10_4: no longer names the net of UC6.11
- net u10_9 renamed CG1_PORT_SELECTED
- net CG1_PORT_SELECTED: now also UD5.3 (1STRB), UD4.12, UD4.6, UD4.9
- net u11_1: no longer names the net of UE7.1, UF8.15 (Q3)
- net u11_13: no longer names the net of UE7.13, UF5.3
- net u11_2: no longer names the net of UE7.2, UF8.11 (~{Q2})
- net u11_5: no longer names the net of UA5.1 (C), UA5.6 (C), UC2.2, UE7.5, UF3.2, UF3.4, UF6.10, UF6.13
- net u11_8: no longer names the net of UD3.7 (Clock_2), UE7.8
- net u12_2: no longer names the net of UC7.6 (~{Q}), UF7.2
- net u12_5 renamed terminal_address_selected
- net terminal_address_selected: no longer UC5.7 (1C)
- net u13_1: no longer names the net of UA6.1
- net u13_1: now also UB1.6; no longer UB6.6
- net u13_12 renamed status_d1
- net status_d1: now also UA9.12
- net u14_3 renamed set_status_d7
- net set_status_d7: now also UB1.3
- net u14_4: no longer names the net of UB5.8 (~{Q})
- net u14_4: now also UB1.4; no longer UB6.4
- net u14_5 renamed unknown_serial_status_bit
- net unknown_serial_status_bit: now also UB1.5
- net u15_10: no longer names the net of UA6.3, UC6.10
- net u15_12: no longer names the net of UC6.12, UF2.6 (~{Q})
- net u15_8 renamed serial_handshake_cts
- net serial_handshake_cts: now also UC9.8
- net u15_9: no longer names the net of UA6.11, UC6.9
- net u16_12: no longer names the net of C25.1, UD6.12 (2RTC)
- net u16_4: no longer names the net of C22.2, UD6.4 (1RTC)
- net u17_12: no longer names the net of C24.2, UE6.12 (2RTC)
- net u17_4: no longer names the net of C23.2, UE6.4 (1RTC)
- net u18_11: no longer names the net of UF6.11, UF8.1 (~{Mr})
- net u18_8: no longer names the net of UF5.9, UF6.8
- net u1_3 renamed single_ended_rts
- net single_ended_rts: no longer R16.1, UD5.1 (1YS_(Pullup))
- net u1_6: no longer names the net of UA8.6 (~{Q})
- net u1_6: now also UD4.10
- net u20_10: no longer names the net of UA6.13, UB5.10 (~{S})
- net u20_2 renamed serial_reg_Q1
- net u20_3 renamed advance_state_machine
- net advance_state_machine: now also UB2.8
- net u22_4: no longer names the net of C26.2
- net u22_4: no longer UD5.4 (1RTC)
- net u24_8: no longer names the net of UF2.13 (~{R}), UF5.8
- net u25_6: no longer names the net of UA4.6 (Serial_Out), UB4.5
- net u25_9: no longer names the net of UA4.9 (Clock)
- net u25_9: no longer UA6.6
- net u27_10 renamed serial_reg_Q7
- net u27_11 renamed serial_reg_Q6
- net u27_12 renamed serial_reg_Q5
- net u27_13 renamed serial_reg_Q4
- net u27_14: no longer names the net of UC4.14 (A=B), UF5.4, UF5.5
- net u27_3 renamed DIP0
- net DIP0: now also SW1.16; no longer SW1.12
- net u27_4 renamed DIP1
- net DIP1: now also SW1.15; no longer SW1.13
- net u27_5 renamed DIP2
- net u27_6 renamed DIP3
- net DIP3: now also SW1.13; no longer SW1.15
- net u27_7 renamed DIP4
- net DIP4: now also SW1.12; no longer SW1.16
- net u27_9 renamed serial_reg_Q8
- net u28_14 renamed status_d0
- net status_d0: now also UA9.2
- net u28_2 renamed status_d7
- net u28_4 renamed status_d6
- net u29_4: no longer names the net of UF4.4 (~{S})
- net u29_4: now also C29.1, R25.2
- net u29_5 renamed unknown_flag_4
- net u2_1: no longer names the net of UC8.6 (~{Q})
- net u2_1: now also UB2.1
- net u2_10: no longer names the net of UE8.15 (Tc)
- net u2_10: now also UB2.10, UD2.9
- net u2_13 renamed n_single_ended_rts
- net n_single_ended_rts: now also UD2.6
- net u2_2: no longer names the net of UC2.4
- net u2_2: now also UB2.2, UB2.4
- net u2_5: no longer names the net of UC8.5 (Q)
- net u2_5: now also UB2.5
- net u2_6: no longer names the net of UA8.13 (~{R})
- net u2_6: now also UB2.6
- net u30_11 renamed serial_out_unknown_flag_3
- net u30_6 renamed serial_register_out
- net u30_9: no longer names the net of UA3.9 (Clock), UA6.8
- net u31_12 renamed serial_reg_Q3
- net serial_reg_Q3: now also UB9.12 (D)
- net u33_12 renamed serial_reg_Q2
- net u34_11 renamed latch_status_d0
- net u34_12: no longer names the net of UA5.15 (Q), UE3.12 (D)
- net u34_13 renamed reset_state_machine
- net reset_state_machine: now also UB1.13, UB1.8, UB9.13 (~{R})
- net u34_2: no longer names the net of UA5.11 (Q), UE3.2 (D)
- net u34_3 renamed latch_status_d1
- net u35_3: no longer names the net of UF3.3
- net u35_3: now also R25.1
- net u35_6: no longer names the net of UC7.10 (~{S}), UF3.6
- net u36_15: no longer names the net of UA2.15 (DO5), UE2.9
- net u36_17: no longer names the net of UA2.17 (DO6), UE2.11
- net u36_19: no longer names the net of UA2.19 (DO7), UE1.1
- net u36_8: no longer names the net of UA2.8 (DO3), UE2.1
- net u37_8: no longer names the net of UC2.8, UE7.3
- net u3_1: no longer names the net of UC8.1 (~{R})
- net u3_1: now also UB1.11
- net u3_10: no longer names the net of UC8.10 (~{S})
- net u3_10: now also UD2.8
- net u3_12 renamed single_ended_data
- net u3_2: no longer names the net of UC8.2 (D), UC8.4 (~{S})
- net u3_3 renamed set_unknown_status_1
- net u3_8: no longer names the net of UC8.8 (~{Q}), UE7.9, UE8.9 (~{Pe})
- net u3_9: no longer names the net of UC8.13 (~{R}), UC8.9 (Q)
- net u40_10: no longer names the net of UA1.10 (DO4), UE1.5
- net u40_15: no longer names the net of UA1.15 (DO5), UD1.9
- net u40_19: no longer names the net of UA1.19 (DO7), UD1.13
- net u40_4: no longer names the net of UA1.4 (DO1), UD1.5
- net u40_6: no longer names the net of UA1.6 (DO2), UD1.3
- net u44_13: no longer names the net of UF1.13 (B)
- net u44_13: now also R23.1; no longer R23.2
- net u44_14: no longer names the net of D1.1 (K), UF1.14 (C)
- net u44_14: now also R1.1, UB1.10; no longer R19.1
- net u44_2: no longer names the net of UF1.2 (B)
- net u44_2: now also R24.2
- net u44_6: no longer names the net of UF1.6 (B)
- net u44_6: now also R19.1
- net u44_8: no longer names the net of R22.1, UF1.8 (C)
- net u44_8: no longer R23.1
- net u44_9: no longer names the net of R20.1, R21.1, UF1.9 (B)
- net u4_11: no longer names the net of UC6.3
- net u4_11: now also UD2.11
- removed net u4_3: R17.1, UA7.9, UD6.15 (2YS_(Pullup)), UE6.15 (2YS_(Pullup)), UE7.10
- net u4_4: no longer names the net of UC8.11 (C), UE8.2 (CK)
- net u4_4: now also UE7.10, UD2.4
- net u6-10: no longer names the net of UF7.4, UF8.10 (Q2)
- net u6-2: no longer names the net of UF6.1, UF8.2 (Q0)
- net u6_12: no longer names the net of UF7.8, UF8.12 (D2)
- net u6_13 renamed address_match_bufd
- net u6_3: no longer names the net of UF5.2, UF8.3 (~{Q0})
- net u6_6: no longer names the net of UF5.1, UF8.6 (~{Q1})
- net u6_7: no longer names the net of UF6.4, UF8.7 (Q1)
- net u7-13 renamed set_status_d6
- net set_status_d6: now also UD4.5; no longer UA7.13
- net u7-2: no longer names the net of UA7.2, UB7.4
- net u7_1: no longer names the net of UA7.1, UA7.4, UB4.1, UB4.3, UB7.10
- net u7_10 renamed status_d5
- net u7_12: no longer names the net of UA6.4, UA7.12
- net u7_5: no longer names the net of UA7.5, UB7.2
- net u7_6: no longer names the net of UA6.10, UA7.6, UF4.10 (~{S})
- net u7_8: no longer names the net of UA6.5, UA6.9, UA7.8
- net u8_11: no longer names the net of UA3.7 (S1), UA4.7 (S1), UB4.10, UB4.4
- net u8_11: no longer UA7.11, UB7.11, UF3.11
- net u8_5: no longer names the net of UB4.8, UB7.5
- net u8_6 renamed serial_out_unknown_flag_1
- net u8_9: no longer names the net of UB4.6, UB7.9
- net u9_1 renamed reset_state_machine_bufd
- net u9_13: no longer names the net of UC7.13 (~{R}), UE7.6
- net u9_9 renamed serial_out_unknown_flag_2
- new net: R4.2, UC1.12 (In5)
- new net: R5.2, UC1.4 (In2)
- new net: R6.1, UC1.14 (In6)
- new net: R7.1, UC1.2 (In1)
- new net: UA9.11, UC9.9
- new net: UA9.13, UB9.10 (~{S})
- new net: UD4.13, UD4.8
- new net: UC2.13, UE7.12
- new net: R17.1, UA7.9
- new net: UA9.3, UC9.10
- new net: R2.2, UC1.10 (In4)
- new net: UC2.11, UF6.3
- new net: UA7.11, UB7.11, UF3.11
- new net: UB1.2, UB2.3
- new net: UB6.4, UB9.8 (~{Q})
- new net: UA9.1, UB6.6
- new net: R3.2, UC1.6 (In3)
- new net: UB2.9, UD2.5
- new net: UC3.1 (M), UC3.2 (N)
- new net: R19.2, R23.2, R24.1
- new net CG1_PIN_D: P15.46 (Pin_46)
- new net CG1_PIN_H: P15.44 (Pin_44)
- new net single_ended_clock: UD2.3, UD6.15 (2YS_(Pullup)), UE6.15 (2YS_(Pullup))
- no-connect marks 88 -> 83
Other:
- note added: "Clock"
- note added: "Data"
- note added: "FIXME"
- note added: "FIXME NO DRIVER"
- note added: "Output shift register buffer"
- note added: "Request to send"
- note added: "bit counter"
- note added: "pulse generator"
- note removed: "/\"
- note removed: "= Data Bus? = Keyboard = Processor Board = Floppy Disk Controller Board (FDC) = RAM Bus = I/O (Duplexer) Board = Printer"
- note removed: "Backplane pins that are not connected to any other pins other than the backplane connector are not connected to the Backplane BUS. Neither are backplane pins whose multi-pin connections are otherwise represented with regular wires"
- note removed: "How to make u4_10 and u12_5 both go high?"
- note removed: "KiCad Bus Range Creator https://bit.ly/KiCadBRC"
- note removed: "Other Trans"
- note removed: "Strobe Input"
- note removed: "UC7A Pin 6 inverse-Q latch"
- note removed: "UF2A pin 5 Q latch"
- note removed: "UF4A Q latch"
- note removed: "UF7A four conditions"
- note removed: "UF8 Pin 10 Q2"
- note removed: "Unused"
- note removed: "WARNING: Until refined & corrected, Global Label tag arrows may not indicate the proper signal in/out direction. IN was used as default when KiCad Symbols (components) were not clear on In vs Out signals, so always check component datasheets when in doubt."
- note removed: "x"
- moved on the sheet: C10, C11, C12, C13, C14, C15, C16, C17, C18, C19, C2, C20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

Commit message: time for pizza
Parts:
- removed unit 1 of UA6
- removed unit 4 of UA6
- removed unit 2 of UB1
- removed unit 2 of UB5
- removed unit 3 of UC6
- renumbered UB2 to UB8, UD4 to UD7, UD2 to UD8
Connections:
- net at UE7.5, UF3.2, UF3.4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: no longer UA5.1 (C), UA5.6 (C), UC2.2, UF6.13
- net at C26.2: now also UD5.4 (1RTC)
- net bit_counter_overflow: now reaches UB8.10, UD8.9, UE8.15 (Tc)
- net bit_counter_overflow: now also UB8.12
- net latch_status_d0 renamed term_selectd_and_S0
- net set_unknown_status_1 renamed n_has_RX'd_16_bits
- new net: UA5.1 (C), UA5.6 (C), UF6.13
- no-connect marks 83 -> 80
Other:
- note added: "0b0000"
- note added: "0b1000 NAND term_select"
- note added: "0bxx00"
- note added: "0bxx1x &term_select &single_ended_rts &_not_was_single_ended_rts"
- note added: "0bxx1x NAND term_selet"
- note added: "0bxxx1 NAND term_seler"
- note added: "AND"
- note added: "seems to be part of enabling serial transmitter"
- note added: "was_single_ended_rts"
- moved on the sheet: UC2E, UF6A, UF6B, UF7A

Commit message: teh cleanup
Parts:
- renumbered UA9 to UA6, UB9 to UB5, UC9 to UC6
Connections:
- net CG1_PIN_N: no longer UC5.3 (1YS), UC5.4 (1YP)
- net D7_out: no longer UC1.3 (~{Out1})
- net single_ended_clock: now also R17.1
- net at UE4.13 (Out6): now also UC1.3 (~{Out1})
- net at UA7.9: no longer R17.1
- net n_single_ended_rts renamed n_has_RX'd_16_bits3
- net u1_8: no longer names the net of UA8.8 (~{Q}), UC6.5
- new net CG1_PIN_C: UC5.3 (1YS), UC5.4 (1YP)
- no-connect marks 80 -> 81
Other:
- note added: "INP Port Access"
- note added: "OUT Port Access"
- note added: "Printer port acess high reg"
- note added: "Printer port acess low reg"
- note added: "Q1 is last bit in"
- note added: "is this a start bit?"
- note added: "ok, i understand this latch now.. it simply waits for the bit overflow then reloads from parallel after seeing the first data bit so i think this is a start bit"
- note removed: "All Points Start and End with Backplane Connector (P15)"
- moved on the sheet: UA8B, UB1A, UB1D, UB2A, UC2C, UC6B, UC8A

Commit message: boop
Parts:
- added R26: 1K, Resistor_THT:R_Axial_DIN0207_L6.3mm_D2.5mm_P10.16mm_Horizontal, symbol SamacSys_Parts:YR1B24K9CC
Connections:
- net XX(UE3P4) is gone; now on net GND: UE3.4 (~{S})
- net u4_12 is gone; now on net CG1_PORT_SELECTED: UC5.9 (CC), UD2.12, UF1.1 (C)
- net CG1_PORT_SELECTED: now also UD6.13 (2STRB); no longer UD7.6, UD7.9
- net D7_out: now also UC1.3 (~{Out1}), UE4.13 (Out6)
- net GND: now also UE3.10 (~{S})
- net VCC: now also UA8.1 (~{R}), R26.2
- net XX(UC7P4): no longer UC7.4 (~{S})
- net single_ended_clock: now also UD5.15 (2YS_(Pullup)), R26.1
- net single_ended_data: no longer R15.1, UD5.15 (2YS_(Pullup))
- net single_ended_rts: now also R15.1, R16.1, UD5.1 (1YS_(Pullup))
- net at UE7.5, UF3.2, UF3.4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: now also UA5.1 (C), UA5.6 (C), UC2.2, UF6.13
- net at UA8.4 (~{S}): now also UA8.13 (~{R}), UB2.6
- net unknown_signal: now reaches UA3.7 (S1), UA4.7 (S1), UB4.10, UB4.4
- net unknown_signal: now also UA7.11, UB7.11, UC7.4 (~{S}), UF3.11
- net /terminal_address_selected: now reaches UC6.12, UF2.6 (~{Q})
- net D6_in9 renamed PERIPHERAL_RESET
- net P15_28 renamed CPU_OUT_0x78
- net P15_32 renamed write_iface_serial_tx_0
- net P15_64 renamed INT_6
- net P15_66 renamed INT_5
- net P15_68 renamed INT_7
- net XX(UB5P11): no longer names the net of UB5.11 (C)
- net XX(UB5P9): no longer names the net of UB5.9 (Q)
- net n_has_RX'd_16_bits renamed N_HAS_RXD_8_BITS
- net n_has_RX'd_16_bits3 renamed n_single_ended_rts
- net read_latch_strobe renamed read_iface_serial_buffer
- net read_printer_status_reg renamed read_iface_prnt_status
- net read_status_latch renamed read_iface_status
- net serial_out_unknown_flag_1: no longer names the net of UA4.11 (D1)
- net serial_out_unknown_flag_1: now also UB7.8; no longer UB7.6
- net serial_out_unknown_flag_3: no longer names the net of UA3.11 (D1)
- net serial_out_unknown_flag_3: now also UB7.6; no longer UB7.8
- net u10_11 renamed ENABLE_CG1_RX
- net unknown_flag_4 renamed terminal_has_data_waiting
- net unknown_serial_status_bit renamed was_selected_and_S1
- new net: UD7.6, UD7.9
- no-connect marks 81 -> 80
Other:
- note added: "0 0 0 1 0"
- note added: "0x02 0b00000010 0x04 0b00001000 0x05 0b00001001 0x06 0b00000110 0x08 0b00001000 0x61 0b01100001 0x40 0b01000000 0x64 0b01100100 0x90 0b10010000"
- note added: "I think this is how we set terminal status of ready"
- note added: "causes the terminal to stop blinking"
- note added: "fixme"
- note added: "is this right?"
- note added: "latch that terminal has data in the serial tx_buffer"
- note added: "lol triggers an interrupt"
- note added: "this latches some state _when_ the terminal is selected with address and S=0x4"
- note added: "this latchis stat wen the terminal is selected with address and S|=0x1"
- note removed: "0bxx1x &term_select &single_ended_rts &_not_was_single_ended_rts"
- note removed: "0bxx1x NAND term_selet"
- note removed: "FIXME NO DRIVER"
- moved on the sheet: C29, R16, R17, R19, R24, R25, UA5A, UA5B, UA6A, UA6D, UA7A, UA7C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

Commit message: borp
Parts:
- removed unit 3 of UB8
- removed unit 3 of UD7
- removed unit 2 of UD7
- removed unit 4 of UD7
- removed unit 3 of UD8
- added unit 3 of UB2
- added unit 3 of UD2
- added unit 2 of UD4
- added unit 4 of UD4
- added unit 3 of UD4
- R1: value 10K -> 330R
- R23: value 330R -> 10K
Connections:
- net XX(UC7P11) is gone; now on net GND: UC7.11 (C)
- net CG1_PIN_D: now also UD5.11 (2B)
- net CG1_PIN_H: now also UD5.9 (2A)
- net CG1_PORT_SELECTED: now also UD4.12
- net D0_out: now also UE4.13 (Out6)
- net D5_in: now also UA5.4 (J)
- net D7_out: no longer UE4.13 (Out6)
- net ENABLE_CG1_RX: now also UD4.11
- net VCC: now also R23.2; no longer R1.2, R16.2
- net advance_state_machine: now also UB2.8
- net bit_counter_overflow: now also UB2.10
- net reset_state_machine: no longer UF2.1 (~{R})
- net single_ended_clock: no longer R26.1, UD5.15 (2YS_(Pullup))
- net single_ended_data: now also R26.1, UD5.15 (2YS_(Pullup))
- net /CPU_OUT_0x78: now reaches UA5.1 (C), UA5.6 (C), UC2.2, UE7.5, UF3.2, UF3.4, UF6.10, UF6.13
- net at UA8.13 (~{R}), UA8.4 (~{S}), UB2.6: now also UA8.9 (Q)
- net at UA8.6 (~{Q}): now also UD4.10
- net POWER_ENABLE: now reaches R22.1, UF1.8 (C)
- net POWER_ENABLE: now also R1.2, R24.1
- net at UF1.13 (B): now also R1.1; no longer R23.1
- net POWER_GOOD: now reaches D1.1 (K), UB1.10, UF1.14 (C)
- net POWER_GOOD: now also R23.1; no longer R1.1
- net at UC6.11: now also UD4.4
- net DIP0 renamed u27_7
- net DIP1 renamed u27_6
- net DIP2 renamed u27_5
- net DIP3 renamed u27_4
- net DIP4 renamed u27_3
- net INT_7 renamed term_selectd_and_S2_INT7
- net XX(UC4P1): no longer names the net of UC4.1 (~{E})
- net latch_status_d1 renamed term_selectd_and_S1
- net n_single_ended_rts renamed /single_ended_rts
- net /single_ended_rts: now also UD2.6
- net set_status_d6 renamed protocol_request_data
- net protocol_request_data: now also UD4.5
- net set_status_d7 renamed 8_bits_from_serial_ready
- net status_d5 renamed /protocol_request_data
- net status_d6 renamed terminal_has_output_data_waiting
- net status_d7 renamed 8_bits_ready_on_latch
- net u4_10 renamed differntial_transmit_enable
- net unknown_signal renamed /term_has_data_when_requested
- new net: UD4.6, UD4.9
- new net: UB2.9, UD2.5
- new net: UD4.13, UD4.8
- new net .8: R19.2
- no-connect marks 80 -> 77
Other:
- note added: ""CG1""
- note added: ""CG2""
- note added: "3 input AND (2 inverted inputs)"
- note added: "any command with this bit as a zero when we have data waiting during a terminal selection, this command alsoo uses the was_single_ended_rts latch"
- note added: "any command with this bit set will INT"
- note added: "causes the terminal to stop blinking- makes sense this just sets a flag for the terminal to read"
- note added: "i believe this sets the required initial state of the CTS an enable are contingent on the state machine being in a receptive state"
- note added: "interface and printer status port access"
- note added: "is wire this right?"
- note added: "this disables CTS if there is no data waiting"
- note added: "this disables the differential RX reciever if we're sending data but only kicks in after a reset"
- note added: "this gate suggests that RTS has to be held LOW? inj order for the 8 bit register latch signal to be recognizd"
- note added: "this just sets a flag for the terminal to read, but no other bits can be set when sending this command"
- note added: "well shit.. didnt see this"
- note removed: "0 0 0 1 0"
- note removed: "Terminal Back I/O Plug "CG1""
- note removed: "Terminal Back I/O Plug "CG2""
- note removed: "causes the terminal to stop blinking"
- note removed: "is this right?"
- note removed: "lol triggers an interrupt"
- note removed: "seems to be part of enabling serial transmitter"
- moved on the sheet: C29, P15, R10, R11, R12, R15, R18, R2, R20, R21, R22, R25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
