File: Trapezoid_Terminal/Backplane/Entrex Trapezoid Backplane v17.kicad_sch (KiCad schematic)
At the start: 18 parts, among them J10 Conn_02x22_Odd_Even, J11 Floppy I/O, J12 Conn_02x15_Odd_Even, J13 Conn_02x15_Odd_Even, J14 Conn_02x15_Odd_Even, J15 Card Edge Connector, J16 Conn_02x50_Odd_Even, J17 trapezoid, J18 Card Edge Connector, J19 trapezoid, J20 trapezoid, J21 Conn_01x07_Pin, J22 Conn_02x12_Odd_Even, J24 Conn_01x08_Pin, J25 Mystery, J9 Conn_02x22_Odd_Even

Commit message: boop
Connections:
- net J17_9 is gone; now on net read_iface_status: J15.10 (Pin_10), J17.9 (Pin_9)
- net J17_11 renamed read_iface_serial_buffer
- net J17_7 renamed read_iface_status
- net J17_71 renamed read_iface_status1
- net J17_72 renamed read_iface_status2
- net J17_75 renamed read_iface_status5
- net J17_78 renamed read_iface_status8
- net J17_79 renamed read_iface_status9
Changed lines of the file:
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@@
     (effects (font (size 1.27 1.27)) (justify left bottom))
   )
-  (label "J17_7" (at 611.505 113.03 0) (fields_autoplaced)
+  (label "read_iface_status" (at 611.505 113.03 0) (fields_autoplaced)
     (effects (font (size 1.27 1.27)) (justify left bottom))
   )
@@
     (effects (font (size 1.27 1.27)) (justify left bottom))
   )
-  (label "J17_78" (at 919.861 348.996 0) (fields_autoplaced)
+  (label "read_iface_status8" (at 919.861 348.996 0) (fields_autoplaced)
     (effects (font (size 1.27 1.27)) (justify left bottom))
   )
@@
     (effects (font (size 1.27 1.27)) (justify left bottom))
   )
-  (label "J17_11" (at 611.505 118.11 0) (fields_autoplaced)
+  (label "read_iface_serial_buffer" (at 611.505 118.11 0) (fields_autoplaced)
     (effects (font (size 1.27 1.27)) (justify left bottom))
   )
@@
     (effects (font (size 1.27 1.27)) (justify left bottom))
   )
-  (label "J17_9" (at 611.505 115.57 0) (fields_autoplaced)
+  (label "read_iface_status" (at 611.505 115.57 0) (fields_autoplaced)
     (effects (font (size 1.27 1.27)) (justify left bottom))
   )
@@
     (effects (font (size 1.27 1.27)) (justify left bottom))
   )
-  (label "J17_9" (at 485.648 119.38 0) (fields_autoplaced)
+  (label "read_iface_status" (at 485.648 119.38 0) (fields_autoplaced)
     (effects (font (size 1.27 1.27)) (justify left bottom))
   )
@@
     (effects (font (size 1.27 1.27)) (justify right bottom))
   )
-  (label "J17_7" (at 485.648 116.84 0) (fields_autoplaced)
+  (label "read_iface_status" (at 485.648 116.84 0) (fields_autoplaced)
     (effects (font (size 1.27 1.27)) (justify left bottom))
   )
@@
     (effects (font (size 1.27 1.27)) (justify left bottom))
   )
-  (label "J17_11" (at 485.648 121.92 0) (fields_autoplaced)
+  (label "read_iface_serial_buffer" (at 485.648 121.92 0) (fields_autoplaced)
     (effects (font (size 1.27 1.27)) (justify left bottom))
   )
@@
     (effects (font (size 1.27 1.27)) (justify left bottom))
   )
-  (label "J17_78" (at 738.759 262.636 0) (fields_autoplaced)
+  (label "read_iface_status8" (at 738.759 262.636 0) (fields_autoplaced)
     (effects (font (size 1.27 1.27)) (justify left bottom))
   )
@@
     )
   )
-  (global_label "J17_11" (shape passive) (at 642.493 118.11 180) (fields_autoplaced)
+  (global_label "read_iface_serial_buffer" (shape passive) (at 642.493 118.11 180) (fields_autoplaced)
     (effects (font (size 1.27 1.27)) (justify right))
     (property "Intersheetrefs" "${INTERSHEET_REFS}" (at 633.9253 118.11 0)
@@
     )
   )
-  (global_label "J17_79" (shape passive) (at 642.493 204.47 180) (fields_autoplaced)
+  (global_label "read_iface_status9" (shape passive) (at 642.493 204.47 180) (fields_autoplaced)
     (effects (font (size 1.27 1.27)) (justify right))
     (property "Intersheetrefs" "${INTERSHEET_REFS}" (at 633.9253 204.47 0)
@@
     )
   )
-  (global_label "J17_75" (shape passive) (at 642.493 199.39 180) (fields_autoplaced)
+  (global_label "read_iface_status5" (shape passive) (at 642.493 199.39 180) (fields_autoplaced)
     (effects (font (size 1.27 1.27)) (justify right))
     (property "Intersheetrefs" "${INTERSHEET_REFS}" (at 633.9253 199.39 0)
@@
     )
   )
-  (global_label "J17_71" (shape passive) (at 642.493 194.31 180) (fields_autoplaced)
+  (global_label "read_iface_status1" (shape passive) (at 642.493 194.31 180) (fields_autoplaced)
     (effects (font (size 1.27 1.27)) (justify right))
     (property "Intersheetrefs" "${INTERSHEET_REFS}" (at 633.9253 194.31 0)
@@
     )
   )
-  (global_label "J17_78" (shape passive) (at 655.193 201.93 0) (fields_autoplaced)
+  (global_label "read_iface_status8" (shape passive) (at 655.193 201.93 0) (fields_autoplaced)
     (effects (font (size 1.27 1.27)) (justify left))
     (property "Intersheetrefs" "${INTERSHEET_REFS}" (at 663.7607 201.93 0)
@@
     )
   )
-  (global_label "J17_11" (shape passive) (at 472.948 121.92 0) (fields_autoplaced)
+  (global_label "read_iface_serial_buffer" (shape passive) (at 472.948 121.92 0) (fields_autoplaced)
     (effects (font (size 1.27 1.27)) (justify left))
     (property "Intersheetrefs" "${INTERSHEET_REFS}" (at 481.5157 121.92 0)
@@
     )
   )
-  (global_label "J17_78" (shape input) (at 940.689 348.996 180) (fields_autoplaced)
+  (global_label "read_iface_status8" (shape input) (at 940.689 348.996 180) (fields_autoplaced)
     (effects (font (size 1.27 1.27)) (justify right))
     (property "Intersheetrefs" "${INTERSHEET_REFS}" (at 931.01 348.996 0)
@@
     )
   )
-  (global_label "J17_7" (shape passive) (at 472.948 116.84 0) (fields_autoplaced)
+  (global_label "read_iface_status" (shape passive) (at 472.948 116.84 0) (fields_autoplaced)
     (effects (font (size 1.27 1.27)) (justify left))
     (property "Intersheetrefs" "${INTERSHEET_REFS}" (at 480.3062 116.84 0)
@@
     )
   )
-  (global_label "J17_72" (shape passive) (at 655.193 194.31 0) (fields_autoplaced)
+  (global_label "read_iface_status2" (shape passive) (at 655.193 194.31 0) (fields_autoplaced)
     (effects (font (size 1.27 1.27)) (justify left))
     (property "Intersheetrefs" "${INTERSHEET_REFS}" (at 663.7607 194.31 0)
@@
     )
   )
-  (global_label "J17_7" (shape passive) (at 642.493 113.03 180) (fields_autoplaced)
+  (global_label "read_iface_status" (shape passive) (at 642.493 113.03 180) (fields_autoplaced)
     (effects (font (size 1.27 1.27)) (justify right))
     (property "Intersheetrefs" "${INTERSHEET_REFS}" (at 635.1348 113.03 0)
@@
     )
   )
-  (global_label "J17_9" (shape passive) (at 472.948 119.38 0) (fields_autoplaced)
+  (global_label "read_iface_status" (shape passive) (at 472.948 119.38 0) (fields_autoplaced)
     (effects (font (size 1.27 1.27)) (justify left))
     (property "Intersheetrefs" "${INTERSHEET_REFS}" (at 480.3062 119.38 0)
@@
     )
   )
-  (global_label "J17_9" (shape passive) (at 642.493 115.57 180) (fields_autoplaced)
+  (global_label "read_iface_status" (shape passive) (at 642.493 115.57 180) (fields_autoplaced)
     (effects (font (size 1.27 1.27)) (justify right))
     (property "Intersheetrefs" "${INTERSHEET_REFS}" (at 635.1348 115.57 0)
